Commit message: feat: extending the limit of ur3e joint by 2*pi when necessary

File: robot/duckify_simulation/urdf/ur3e.urdf (robot description, URDF)
Before this commit: robot ur3e, 16 links, 15 joints
Joints:
- joint elbow_joint: limit lower=-3.141592653589793 upper=3.141592653589793 effort=28.0 velocity=3.141592653589793 -> lower=-6.283185307179586 upper=6.283185307179586 effort=28.0 velocity=3.141592653589793

Commit message: fix: various labo fix on the filter and collisions, and the 180 degree flip

File: robot/duckify_simulation/urdf/ur3e.urdf (robot description, URDF)
Before this commit: robot ur3e, 16 links, 15 joints
Joints:
- joint pen_joint: origin xyz=0 0 0.1051 rpy=3.141592653589793 0 0 -> xyz=0 0 0.1031 rpy=3.141592653589793 0 0
